File: Hardware/LiPoBBSupplyWithCharging.brd (EAGLE design)
At the start: 55 x 15.2 mm, 30 parts

Commit message: updates
Parts:
- removed C9: 4.7u, CalvEngIO-Passives:C0603
- removed SWITCH1: SWITCH.JS202011JCQN, CalvEngIO-Switches:SWITCH.00
- added C8: 2.2u, CalvEngIO-Passives:C0603
- added SWITCH: SWITCH.JS202011JCQN, CalvEngIO-Switches:SWITCH.00
- C1, C2, C4, C5: value 4.7u -> 2.2u
- D3, D4: device CalvEngIO-DiscreteSemi:SOD-323 -> CalvEngIO-DiscreteSemi:USC
- R4: value (none) -> 10k
- USB: value USB.MICRO -> USB.MICRO.PWR-BIGGERPADS; device CalvEngIO-Connectors:USB-MICRO-01 -> CalvEngIO-Connectors:USB-MICRO-01.BIGGERPADS.PWR
- moved C7 23.9 mm to (37.5, 2.77), turned to 90 degrees
- moved LOGO1 18.3 mm to (5.51, 13.0)
- moved D4 0.33 mm to (24.6, 7.92), turned to 180 degrees
- moved D3 0.10 mm to (16.9, 4.60), turned to 90 degrees
- renumbered LIPO1 to LIPO, R5 to R3, R7 to R2, VDD to PWR
Connections:
- removed net N$13: USB.3
- removed net N$17: USB.2
- net GND: now also C8.2; no longer C9.2
- net N$9: now also D3.-, D4.-, SWITCH.2; no longer D3.C, D4.C, SWITCH1.2
- net VIN: now also C7.1, SWITCH.3; no longer C9.1, SWITCH1.3
- net VLIPO: now also C8.1, D3.+; no longer C7.1, D3.A
- net V_USB: now also D4.+; no longer D4.A
Routing:
- net VLIPO: track 36.9 -> 41.4 mm
- net VIN: track 36.3 -> 37.4 mm
- net GND: track 22.8 -> 23.6 mm
Other:
- board text added: "LiPo Battery Breadboard Power Supply with Charging"
- board text added: "Rev C"
- board text removed: "Rev A"
