File: Hardware/LiPoBBSupplyWithCharging.sch (EAGLE design)
At the start: 30 parts

Commit message: updates
Parts:
- removed C9: 4.7u, CalvEngIO-Passives:CAPACITOR0603
- added C8: 2.2u, CalvEngIO-Passives:CAPACITOR0603
- C1, C2, C4, C5: value 4.7u -> 2.2u
- D3, D4: device CalvEngIO-DiscreteSemi:DIODE-BAS16J -> CalvEngIO-DiscreteSemi:SCHOTTKY-USC
- R4: value (none) -> 10k
- USB: value USB.MICRO -> USB.MICRO.PWR-BIGGERPADS; device CalvEngIO-Connectors:USB.MICRO -> CalvEngIO-Connectors:USB.MICRO.PWR-BIGGERPADS
- renumbered LIPO1 to LIPO, R5 to R3, R7 to R2, SWITCH1 to SWITCH, VDD to PWR
Connections:
- removed net N$13: USB.D+
- removed net N$17: USB.D-
- net GND: now also C8.2; no longer C9.2
- net VIN: now also C7.1; no longer C9.1
- net VLIPO: now also C8.1; no longer C7.1
Other:
- note added: "Rev E"
- note removed: "Rev A"
- moved on the sheet: C7
